Commit message: added some surfaces for contacts + scaled small urdf

File: urdf/human.urdf (robot description, URDF)
Before this commit: robot HUMAN, 66 links, 65 joints
Links:
- link HipsLink: geometry collision mesh filename=package://human_description/meshes/HipsLinkFull.dae scale=1 1 0.8; visual mesh filename=package://human_description/meshes/HipsLinkFull.dae scale=1 1 0.8
- link LArmLink: geometry collision mesh filename=package://human_description/meshes/LArmLinkFull.dae scale=1 1 1; visual mesh filename=package://human_description/meshes/LArmLinkFull.dae scale=1 1 1
- link LForearmLink: geometry collision mesh filename=package://human_description/meshes/LForearmLink.dae scale=1 1 0.875; visual mesh filename=package://human_description/meshes/LForearmLink.dae scale=1 1 0.875
- link LLegLink: geometry collision mesh filename=package://human_description/meshes/LLegLink.dae scale=1 1 1; visual mesh filename=package://human_description/meshes/LLegLink.dae scale=1 1 1
- link LShinLink: geometry collision mesh filename=package://human_description/meshes/LShinLink.dae scale=1 1 1; visual mesh filename=package://human_description/meshes/LShinLink.dae scale=1 1 1
- link RArmLink: geometry collision mesh filename=package://human_description/meshes/RArmLinkFull.dae scale=1 1 1; visual mesh filename=package://human_description/meshes/RArmLinkFull.dae scale=1 1 1
- link RForearmLink: geometry collision mesh filename=package://human_description/meshes/RForearmLink.dae scale=1 1 0.875; visual mesh filename=package://human_description/meshes/RForearmLink.dae scale=1 1 0.875
- link RLegLink: geometry collision mesh filename=package://human_description/meshes/RLegLink.dae scale=1 1 1; visual mesh filename=package://human_description/meshes/RLegLink.dae scale=1 1 1
- link RShinLink: geometry collision mesh filename=package://human_description/meshes/RShinLink.dae scale=1 1 1; visual mesh filename=package://human_description/meshes/RShinLink.dae scale=1 1 1
- link TorsoLink: geometry collision mesh filename=package://human_description/meshes/TorsoLinkFull.dae scale=1 1 0.9; visual mesh filename=package://human_description/meshes/TorsoLinkFull.dae scale=1 1 0.9
Joints:
- joint Head_0: origin xyz=-0.025 0.0 0.525 rpy=0.0 0.0 0.0 -> xyz=-0.025 0.0 0.46 rpy=0.0 0.0 0.0
- joint LAnkle_0: origin xyz=-0.025 0.0 -0.375 rpy=0.0 0.0 0.0 -> xyz=-0.025 0.0 -0.37 rpy=0.0 0.0 0.0
- joint LArm_0: limit lower=-1.42 upper=1.57 effort=100 velocity=100 -> lower=-1.42 upper=1.57 effort=60 velocity=100; origin xyz=-0.05 0.15 0.35 rpy=0.0 0.0 0.0 -> xyz=-0.05 0.15 0.30 rpy=0.0 0.0 0.0
- joint LLeg_0: origin xyz=-0.0 0.1 -0.15 rpy=0.0 0.0 0.0 -> xyz=-0.0 0.1 -0.1 rpy=0.0 0.0 0.0
- joint LLeg_1: limit lower=-2.3 upper=0.52 effort=100 velocity=100 -> lower=-2.3 upper=0.52 effort=60 velocity=100
- joint LShin_0: limit lower=0.0 upper=2.6 effort=100 velocity=100 -> lower=0.0 upper=2.6 effort=60 velocity=100
- joint LWrist_0: origin xyz=0.01 0.24 -0.01 rpy=0.0 0.0 0.0 -> xyz=0.01 0.21 -0.01 rpy=0.0 0.0 0.0
- joint RAnkle_0: origin xyz=-0.025 0.0 -0.375 rpy=0.0 0.0 0.0 -> xyz=-0.025 0.0 -0.37 rpy=0.0 0.0 0.0
- joint RArm_0: limit lower=-1.42 upper=1.57 effort=100 velocity=100 -> lower=-1.42 upper=1.57 effort=60 velocity=100; origin xyz=-0.05 -0.15 0.35 rpy=0.0 0.0 0.0 -> xyz=-0.05 -0.15 0.3 rpy=0.0 0.0 0.0
- joint RLeg_0: origin xyz=-0.0 -0.1 -0.15 rpy=0.0 0.0 0.0 -> xyz=-0.0 -0.1 -0.1 rpy=0.0 0.0 0.0
- joint RLeg_1: limit lower=-2.3 upper=0.52 effort=100 velocity=100 -> lower=-2.3 upper=0.52 effort=60 velocity=100
- joint RShin_0: limit lower=0.0 upper=2.6 effort=100 velocity=100 -> lower=0.0 upper=2.6 effort=60 velocity=100
- joint RWrist_0: origin xyz=0.01 -0.24 -0.01 rpy=0.0 0.0 0.0 -> xyz=0.01 -0.21 -0.01 rpy=0.0 0.0 0.0

Commit message: Restore original values for dynamic rescale and add elbow joint

File: urdf/human.urdf (robot description, URDF)
Before this commit: robot HUMAN, 66 links, 65 joints
Links:
- added link elbow2lforearm, mass 0.05
- added link elbow2rforearm, mass 0.05
- link HipsLink: geometry collision mesh filename=package://human_description/meshes/HipsLinkFull.dae scale=1 1 1; visual mesh filename=package://human_description/meshes/HipsLinkFull.dae scale=1 1 1
- link LForearmLink: geometry collision mesh filename=package://human_description/meshes/LForearmLink.dae scale=1 1 1; visual mesh filename=package://human_description/meshes/LForearmLink.dae scale=1 1 1
- link RForearmLink: geometry collision mesh filename=package://human_description/meshes/RForearmLink.dae scale=1 1 1; visual mesh filename=package://human_description/meshes/RForearmLink.dae scale=1 1 1
- link TorsoLink: geometry collision mesh filename=package://human_description/meshes/TorsoLinkFull.dae scale=1 1 1; visual mesh filename=package://human_description/meshes/TorsoLinkFull.dae scale=1 1 1
Joints:
- removed joint LForearm
- removed joint RForearm
- added joint LForearm_0: type revolute, parent LElbowLink, child elbow2lforearm, origin xyz=-0.01 0.05 0.0 rpy=0.0 0.0 0.0, axis 0 0 1, limit lower=-2.5 upper=0.0 effort=100 velocity=100
- added joint LForearm_1: type revolute, parent elbow2lforearm, child LForearmLink, origin xyz=-0.01 0.05 0.0 rpy=0.0 0.0 0.0, axis 0 1 0, limit lower=-1.57 upper=1.0 effort=100 velocity=100
- added joint RForearm_0: type revolute, parent RElbowLink, child elbow2rforearm, origin xyz=-0.01 -0.05 0.0 rpy=0.0 0.0 0.0, axis 0 0 1, limit lower=0.0 upper=2.5 effort=100 velocity=100
- added joint RForearm_1: type revolute, parent elbow2rforearm, child RForearmLink, origin xyz=-0.01 -0.05 0.0 rpy=0.0 0.0 0.0, axis 0 1 0, limit lower=-1.57 upper=1.0 effort=100 velocity=100
- joint Head_0: origin xyz=-0.025 0.0 0.46 rpy=0.0 0.0 0.0 -> xyz=-0.025 0.0 0.525 rpy=0.0 0.0 0.0
- joint LAnkle_0: origin xyz=-0.025 0.0 -0.37 rpy=0.0 0.0 0.0 -> xyz=-0.025 0.0 -0.375 rpy=0.0 0.0 0.0
- joint LArm_0: origin xyz=-0.05 0.15 0.30 rpy=0.0 0.0 0.0 -> xyz=-0.05 0.15 0.35 rpy=0.0 0.0 0.0
- joint LElbow: axis 0 1 0 -> (none); limit lower=-1.57 upper=1.0 effort=100 velocity=100 -> (none); type revolute -> fixed
- joint LLeg_0: origin xyz=-0.0 0.1 -0.1 rpy=0.0 0.0 0.0 -> xyz=-0.0 0.1 -0.15 rpy=0.0 0.0 0.0
- joint LWrist_0: origin xyz=0.01 0.21 -0.01 rpy=0.0 0.0 0.0 -> xyz=0.01 0.24 -0.01 rpy=0.0 0.0 0.0
- joint RAnkle_0: origin xyz=-0.025 0.0 -0.37 rpy=0.0 0.0 0.0 -> xyz=-0.025 0.0 -0.375 rpy=0.0 0.0 0.0
- joint RArm_0: origin xyz=-0.05 -0.15 0.3 rpy=0.0 0.0 0.0 -> xyz=-0.05 -0.15 0.35 rpy=0.0 0.0 0.0
- joint RElbow: axis 0 1 0 -> (none); limit lower=-1.57 upper=1.0 effort=100 velocity=100 -> (none); type revolute -> fixed
- joint RLeg_0: origin xyz=-0.0 -0.1 -0.1 rpy=0.0 0.0 0.0 -> xyz=-0.0 -0.1 -0.15 rpy=0.0 0.0 0.0
- joint RWrist_0: origin xyz=0.01 -0.21 -0.01 rpy=0.0 0.0 0.0 -> xyz=0.01 -0.24 -0.01 rpy=0.0 0.0 0.0
